File: kicad/easyplc.sch (KiCad schematic (older format))
At the start: 41 parts, among them P1 RELAYS, P10 COMMS, P11 ADC L, P12 ADC H, P13 Reset, P14 MICROSD, P15 GO SW, P2 STOPSW, P3 RS485, P4 MODBUS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

Commit message: Download support added.  Debugging 2nd axis code.
Parts:
- removed R1, R2, R4, R5: 1k, symbol R
- added P16: EXT POWER, symbol CONN_4
- P1: symbol CONN_5X2 -> CONN_4X2
Connections:
- net +24V: now also P16.1 (P1); no longer P1.2
- net +5V: now also P16.4 (P4)
- net DIG24: no longer P2.2
- net DIG25: now also P2.2
- net DIG26: no longer P2.4
- net DIG27: now also P2.4
- net DIG28: no longer P2.6
- net DIG29: now also P2.6
- net DIG30: no longer P2.8
- net DIG31: now also P2.8
- net DIG32: no longer R14.1
- net DIG33: now also R14.1
- net DIG34: no longer R12.1
- net DIG35: now also R12.1
- net DIG36: no longer R7.1
- net DIG37: now also R7.1
- net DIG38: no longer R3.1
- net DIG39: now also R3.1
- net DIG40: no longer P15.2 (PM)
- net DIG41: now also P15.2 (PM)
- net GND: now also P16.2 (P2), P16.3 (P3); no longer P1.9
- net at Q4.E, R15.2: now also P1.2; no longer P1.10
- net at Q1.E, R6.2: now also P1.8; no longer P1.4
- net at Q3.E, R13.2: now also P1.4; no longer P1.8
- net +3.3V: no longer names the net of P9.2
- no-connect marks 0 -> 56
